File: ManiAmpPCB/ManiAmpPCB.kicad_sch (KiCad schematic)
At the start: 28 parts, among them U1 ADAU1701, U2 TPA3116D2DAD, U3 TPA3116D2DAD

Commit message: Schematics WIP
Parts:
- added C17, C18, C19, C20: 220 nF, symbol Device:C
- added C21, C22, C23, C24: 680 nF, symbol Device:C
- added C25, C26, C27, C28: 1 nF, symbol Device:C
- added C29, C30, C31, C32: 10 nF, symbol Device:C
- added C33: 1n, symbol Device:C
- added C34, C37: 220 u, symbol Device:C_Polarized
- added C35, C36: 100 n, symbol Device:C
- added C38, C39, C40: 1 u, symbol Device:C
- added J1, J2, J3, J4: Screw_Terminal_01x02, symbol Connector:Screw_Terminal_01x02
- added JP10, JP2, JP3, JP4, JP5, JP6, JP7, JP8, JP9: SolderJumper_2_Open, symbol Jumper:SolderJumper_2_Open
- added L5, L6, L7, L8: 10 uH, symbol Device:L
- added R10: 100 k, symbol Device:R
- added R11: 20 k, symbol Device:R
- added R5: 10 k, symbol Device:R
- added R6, R7, R8, R9: 3.3 R, symbol Device:R
Connections:
- net GND: now also U2.13 (AM2), U2.14 (AM1), U2.15 (AM0), C21.2, C22.1, C23.2, C24.1, C25.2, C26.1, C27.2, C28.1, C29.2, C30.1, C31.2, C32.1, C33.2, C34.2, C35.2, C36.2, C37.2, C38.2, R11.2
- net at C3.2, L1.1, U2.23 (OUTPL): now also JP1.2 (B)
- net at C14.2, C8.2, L4.2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: now also J2.2 (Pin_2)
- net at U2.16 (SYNC): now also R5.1
- net PVCC: now reaches U2.17 (AVCC)
- net PVCC: now also U2.18 (PVCC_18), U2.19 (PVCC_19), U2.31 (PVCC_31), U2.32 (PVCC_32), C34.1, C35.1, C36.1, C37.1
- net at C4.2, U2.21 (OUTNL): now also JP1.1 (A), JP2.2 (B); no longer L2.1
- net at C2.2, U2.27 (OUTNR): now also JP3.1 (A), JP4.2 (B); no longer L4.1
- net at C1.2, L3.1, U2.29 (OUTPR): now also JP3.2 (B), JP5.1 (A)
- net at U2.6 (PLIMIT): now also U2.7 (GVDD), C38.1, R10.1
- net at U2.8 (GAIN/SLV): now also R10.2, R11.1
- net at C5.1, C9.1, L1.2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: now also J1.1 (Pin_1)
- net at C13.1, C7.1, L3.2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: now also J2.1 (Pin_1)
- net at C10.2, C6.2, L2.2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: now also J1.2 (Pin_2)
- net at U3.16 (SYNC): now also C33.1, R5.2
- net at U3.20 (BSNL): now also C20.1
- net at U3.21 (OUTNL): now also C20.2, JP6.1 (A), JP7.2 (B)
- net at U3.23 (OUTPL): now also C18.2, JP6.2 (B), L5.1
- net at U3.24 (BSPL): now also C18.1
- net at U3.26 (BSNR): now also C19.1
- net at U3.27 (OUTNR): now also C19.2, JP10.2 (B), JP9.1 (A)
- net at U3.29 (OUTPR): now also C17.2, JP8.1 (A), JP9.2 (B), L7.1
- net at U3.30 (BSPR): now also C17.1
- net at U3.6 (PLIMIT): now also U3.7 (GVDD)
- new net: JP10.1 (A), L8.1
- new net: C21.1, C25.1, J3.1 (Pin_1), L5.2, R6.1
- new net: C29.1, R6.2
- new net: C23.1, C27.1, J4.1 (Pin_1), L7.2, R8.1
- new net: C24.2, C28.2, J4.2 (Pin_2), L8.2, R9.2
- new net: C22.2, C26.2, J3.2 (Pin_2), L6.2, R7.2
- new net: JP4.1 (A), L4.1
- new net: C30.2, R7.1
- new net: JP7.1 (A), JP8.2 (B), L6.1
- new net: C32.2, R9.1
- new net: JP2.1 (A), JP5.2 (B), L2.1
- new net: C31.1, R8.2
Other:
- moved on the sheet: C13, C14, C15, C16, C7, C8, JP1, L1, L2, L3, L4, R3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

Commit message: DSP schematics WiP
Parts:
- removed C1, C17, C18, C19, C2, C20, C3, C4: 220 nF, symbol Device:C
- removed C10, C13, C14, C25, C26, C27, C28, C9: 1 nF, symbol Device:C
- removed C11, C12, C15, C16, C29, C30, C31, C32: 10 nF, symbol Device:C
- removed C21, C22, C23, C24, C5, C6, C7, C8: 680 nF, symbol Device:C
- removed C33: 1n, symbol Device:C
- removed C34, C37: 220 u, symbol Device:C_Polarized
- removed C35, C36: 100 n, symbol Device:C
- removed C38, C39, C40: 1 u, symbol Device:C
- removed J1, J2, J3, J4: Screw_Terminal_01x02, symbol Connector:Screw_Terminal_01x02
- removed JP1, JP10, JP2, JP3, JP4, JP5, JP6, JP7, JP8, JP9: SolderJumper_2_Open, symbol Jumper:SolderJumper_2_Open
- removed L1, L2, L3, L4, L5, L6, L7, L8: 10 uH, symbol Device:L
- removed R1, R2, R3, R4, R6, R7, R8, R9: 3.3 R, symbol Device:R
- removed R10: 100 k, symbol Device:R
- removed R11: 20 k, symbol Device:R
- removed R5: 10 k, symbol Device:R
- removed U1: ADAU1701, Package_QFP:LQFP-48_7x7mm_P0.5mm, symbol DSP_AnalogDevices:ADAU1701
- removed U2, U3: TPA3116D2DAD, TPA3116D2DAD:SOP65P810X115-32N, symbol Manifold:TPA3116D2DAD
Other:
- added sheet Amplifier (Amp.kicad_sch)
- added sheet Controller (esp.kicad_sch)
- added sheet DSP (dsp.kicad_sch)
- added sheet Power cascade (power.kicad_sch)

Commit message: Schematics WiP
Other:
- sheet DSP renamed Audio processing
- sheet Audio processing: file dsp.kicad_sch -> audio_processing.kicad_sch
Changed lines of the file:
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@@
     (instances
       (project "ManiAmpPCB"
-        (path "/68848034-b876-4050-8b11-378a17137257" (page "5"))
+        (path "/68848034-b876-4050-8b11-378a17137257" (page "3"))
       )
     )
@@
     (instances
       (project "ManiAmpPCB"
-        (path "/68848034-b876-4050-8b11-378a17137257" (page "4"))
+        (path "/68848034-b876-4050-8b11-378a17137257" (page "5"))
       )
     )
@@
     (stroke (width 0.1524) (type solid))
     (fill (color 0 0 0 0.0000))
-    (property "Sheetname" "DSP" (at 180.34 135.1784 0)
+    (property "Sheetname" "Audio processing" (at 180.34 135.1784 0)
       (effects (font (size 1.27 1.27)) (justify left bottom))
     )
-    (property "Sheetfile" "dsp.kicad_sch" (at 180.34 164.4146 0)
+    (property "Sheetfile" "audio_processing.kicad_sch" (at 180.34 164.4146 0)
       (effects (font (size 1.27 1.27)) (justify left top))
     )
     (instances
       (project "ManiAmpPCB"
-        (path "/68848034-b876-4050-8b11-378a17137257" (page "2"))
+        (path "/68848034-b876-4050-8b11-378a17137257" (page "4"))
       )
     )
