File: ManiAmpPCB/dsp.kicad_sch (KiCad schematic)
At the start: 43 parts, among them Q1 MMBT3906, U1 ADAU1701, U4 AP1117-33, Y1 12.228 MHz

Commit message: Schematics WiP
Parts:
- added U9: INA134UA, INA134UA:SOIC127P599X175-8N, symbol INA134UA:INA134UA
Changed lines of the file:
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@@
       (effects (font (size 1.27 1.27)) hide)
     )
-    (pin "2")
-    (pin "1")
+    (pin "1")
+    (pin "2")
     (instances
       (project "ManiAmpPCB"
@@
       (effects (font (size 1.27 1.27)) hide)
     )
-    (pin "2")
-    (pin "1")
+    (pin "1")
+    (pin "2")
     (instances
       (project "ManiAmpPCB"
@@
       (effects (font (size 1.27 1.27)) hide)
     )
-    (pin "2")
-    (pin "1")
+    (pin "1")
+    (pin "2")
     (instances
       (project "ManiAmpPCB"
@@
       (effects (font (size 1.27 1.27)) hide)
     )
-    (pin "2")
-    (pin "1")
+    (pin "1")
+    (pin "2")
     (instances
       (project "ManiAmpPCB"
@@
       (effects (font (size 1.27 1.27)) hide)
     )
-    (pin "2")
-    (pin "1")
+    (pin "1")
+    (pin "2")
     (instances
       (project "ManiAmpPCB"
@@
       (effects (font (size 1.27 1.27)) (justify left) hide)
     )
+    (pin "1")
+    (pin "2")
     (pin "3")
-    (pin "2")
-    (pin "1")
     (instances
       (project "ManiAmpPCB"
@@
       (effects (font (size 1.27 1.27)) hide)
     )
-    (pin "2")
-    (pin "1")
+    (pin "1")
+    (pin "2")
     (instances
       (project "ManiAmpPCB"
@@
     )
   )
+  (symbol (lib_id "INA134UA:INA134UA") (at 62.23 132.08 0) (unit 1)
+    (in_bom yes) (on_board yes) (dnp no) (fields_autoplaced)
+    (property "Reference" "U9" (at 62.23 114.3 0)
+      (effects (font (size 1.27 1.27)))
+    )
+    (property "Value" "INA134UA" (at 62.23 116.84 0)
+      (effects (font (size 1.27 1.27)))
+    )
+    (property "Footprint" "INA134UA:SOIC127P599X175-8N" (at 62.23 132.08 0)
+      (effects (font (size 1.27 1.27)) (justify bottom) hide)
+    )
+    (property "Datasheet" "" (at 62.23 132.08 0)
+      (effects (font (size 1.27 1.27)) hide)
+    )
+    (property "MF" "Texas Instruments" (at 62.23 132.08 0)
+      (effects (font (size 1.27 1.27)) (justify bottom) hide)
+    )
+    (property "Description" "\nSingle, Audio Differential Line Receivers, 0dB (G=1)\n" (at 62.23 132.08 0)
+      (effects (font (size 1.27 1.27)) (justify bottom) hide)
+    )
+    (property "Package" "SOIC-8 Texas Instruments" (at 62.23 132.08 0)
+      (effects (font (size 1.27 1.27)) (justify bottom) hide)
+    )
+    (property "Price" "None" (at 62.23 132.08 0)
+      (effects (font (size 1.27 1.27)) (justify bottom) hide)
+    )
+    (property "SnapEDA_Link" "https://www.snapeda.com/parts/INA134UA/Texas+Instruments/view-part/?ref=snap" (at 62.23 132.08 0)
+      (effects (font (size 1.27 1.27)) (justify bottom) hide)
+    )
+    (property "MP" "INA134UA" (at 62.23 132.08 0)
+      (effects (font (size 1.27 1.27)) (justify bottom) hide)
+    )
+    (property "Purchase-URL" "https://www.snapeda.com/api/url_track_click_mouser/?unipart_id=10479&manufacturer=Texas Instruments&part_name=INA134UA&search_term=ina134" (at 62.23 132.08 0)
+      (effects (font (size 1.27 1.27)) (justify bottom) hide)
+    )
+    (property "Availability" "In Stock" (at 62.23 132.08 0)
+      (effects (font (size 1.27 1.27)) (justify bottom) hide)
+    )
+    (property "Check_prices" "https://www.snapeda.com/parts/INA134UA/Texas+Instruments/view-part/?ref=eda" (at 62.23 132.08 0)
+      (effects (font (size 1.27 1.27)) (justify bottom) hide)
+    )
+    (pin "1")
+    (pin "2")
+    (pin "3")
+    (pin "4")
+    (pin "5")
+    (pin "6")
+    (pin "7")
+    (instances
+      (project "ManiAmpPCB"
+        (path "/68848034-b876-4050-8b11-378a17137257/f078a227-be2b-4508-9004-00ac4b51165b"
+          (reference "U9") (unit 1)
+        )
+      )
+    )
+  )
   (symbol (lib_id "Device:R") (at 232.41 102.87 90) (unit 1)
     (in_bom yes) (on_board yes) (dnp no)
@@
       (effects (font (size 1.27 1.27)) hide)
     )
-    (pin "2")
-    (pin "1")
+    (pin "1")
+    (pin "2")
     (instances
       (project "ManiAmpPCB"
@@
       (effects (font (size 1.27 1.27)) hide)
     )
-    (pin "2")
-    (pin "1")
+    (pin "1")
+    (pin "2")
     (instances
       (project "ManiAmpPCB"
@@
       (effects (font (size 1.27 1.27)) hide)
     )
-    (pin "26")
-    (pin "33")
-    (pin "21")
-    (pin "38")
-    (pin "48")
-    (pin "6")
-    (pin "39")
-    (pin "7")
-    (pin "23")
-    (pin "45")
-    (pin "3")
-    (pin "22")
-    (pin "30")
-    (pin "16")
-    (pin "24")
-    (pin "44")
-    (pin "43")
-    (pin "27")
-    (pin "25")
-    (pin "9")
-    (pin "28")
-    (pin "36")
-    (pin "5")
-    (pin "8")
-    (pin "35")
-    (pin "37")
-    (pin "46")
-    (pin "47")
-    (pin "17")
-    (pin "18")
-    (pin "2")
-    (pin "19")
-    (pin "1")
-    (pin "31")
-    (pin "20")
-    (pin "32")
-    (pin "40")
-    (pin "29")
-    (pin "34")
-    (pin "4")
+    (pin "1")
     (pin "10")
     (pin "11")
@@
     (pin "14")
     (pin "15")
+    (pin "16")
+    (pin "17")
+    (pin "18")
+    (pin "19")
+    (pin "2")
+    (pin "20")
+    (pin "21")
+    (pin "22")
+    (pin "23")
+    (pin "24")
+    (pin "25")
+    (pin "26")
+    (pin "27")
+    (pin "28")
+    (pin "29")
+    (pin "3")
+    (pin "30")
+    (pin "31")
+    (pin "32")
+    (pin "33")
+    (pin "34")
+    (pin "35")
+    (pin "36")
+    (pin "37")
+    (pin "38")
+    (pin "39")
+    (pin "4")
+    (pin "40")
+    (pin "41")
     (pin "42")
-    (pin "41")
+    (pin "43")
+    (pin "44")
+    (pin "45")
+    (pin "46")
+    (pin "47")
+    (pin "48")
+    (pin "5")
+    (pin "6")
+    (pin "7")
+    (pin "8")
+    (pin "9")
     (instances
       (project "ManiAmpPCB"
@@
       (effects (font (size 1.27 1.27)) hide)
     )
-    (pin "2")
-    (pin "1")
+    (pin "1")
+    (pin "2")
     (instances
       (project "ManiAmpPCB"
@@
       (effects (font (size 1.27 1.27)) hide)
     )
-    (pin "2")
-    (pin "1")
+    (pin "1")
+    (pin "2")
     (instances
       (project "ManiAmpPCB"
@@
       (effects (font (size 1.27 1.27)) hide)
     )
-    (pin "2")
-    (pin "1")
+    (pin "1")
+    (pin "2")
     (instances
       (project "ManiAmpPCB"
@@
       (effects (font (size 1.27 1.27)) hide)
     )
-    (pin "2")
-    (pin "1")
+    (pin "1")
+    (pin "2")
     (instances
       (project "ManiAmpPCB"
@@
       (effects (font (size 1.27 1.27)) hide)
     )
-    (pin "2")
-    (pin "1")
+    (pin "1")
+    (pin "2")
     (instances
       (project "ManiAmpPCB"
@@
       (effects (font (size 1.27 1.27)) hide)
     )
-    (pin "2")
-    (pin "1")
+    (pin "1")
+    (pin "2")
     (instances
       (project "ManiAmpPCB"
@@
       (effects (font (size 1.27 1.27)) hide)
     )
-    (pin "2")
-    (pin "1")
+    (pin "1")
+    (pin "2")
     (instances
       (project "ManiAmpPCB"
@@
       (effects (font (size 1.27 1.27)) hide)
     )
-    (pin "2")
-    (pin "1")
+    (pin "1")
+    (pin "2")
     (instances
       (project "ManiAmpPCB"
@@
       (effects (font (size 1.27 1.27)) hide)
     )
-    (pin "2")
-    (pin "1")
+    (pin "1")
+    (pin "2")
     (instances
       (project "ManiAmpPCB"
@@
       (effects (font (size 1.27 1.27)) hide)
     )
-    (pin "2")
-    (pin "1")
+    (pin "1")
+    (pin "2")
     (instances
       (project "ManiAmpPCB"
@@
       (effects (font (size 1.27 1.27)) hide)
     )
-    (pin "2")
-    (pin "1")
+    (pin "1")
+    (pin "2")
     (instances
       (project "ManiAmpPCB"
@@
       (effects (font (size 1.27 1.27)) hide)
     )
-    (pin "2")
-    (pin "1")
+    (pin "1")
+    (pin "2")
     (instances
       (project "ManiAmpPCB"
@@
       (effects (font (size 1.27 1.27)) hide)
     )
-    (pin "2")
-    (pin "1")
+    (pin "1")
+    (pin "2")
     (instances
       (project "ManiAmpPCB"
@@
       (effects (font (size 1.27 1.27)) hide)
     )
-    (pin "2")
-    (pin "1")
+    (pin "1")
+    (pin "2")
     (instances
       (project "ManiAmpPCB"
@@
       (effects (font (size 1.27 1.27)) hide)
     )
-    (pin "2")
-    (pin "1")
+    (pin "1")
+    (pin "2")
     (instances
       (project "ManiAmpPCB"
@@
       (effects (font (size 1.27 1.27)) hide)
     )
+    (pin "1")
+    (pin "2")
     (pin "3")
-    (pin "2")
-    (pin "1")
-    (instances
-      (project "ManiAmpPCB"
+    (instances
+      (project "ManiAmpPCB"
