File: ManiAmpPCB/esp.kicad_sch (KiCad schematic)
At the start: 0 parts

Commit message: Schematics WiP
Parts:
- added C85, C87: 22 uF, Capacitor_SMD:C_0805_2012Metric, symbol Device:C
- added C86, C88, C89, C91, C92: 100 nF, Capacitor_SMD:C_0603_1608Metric, symbol Device:C
- added C90: 2.2 uF, Capacitor_SMD:C_0603_1608Metric, symbol Device:C
- added C93: 10 uF, Capacitor_SMD:C_0603_1608Metric, symbol Device:C
- added C94, C95: 100 n, Capacitor_SMD:C_0603_1608Metric, symbol Device:C
- added D3, D4: 1N5711, Diode_SMD:D_SOD-123, symbol Diode:1N5711
- added J6: Prog, Connector_PinHeader_2.54mm:PinHeader_2x03_P2.54mm_Vertical, symbol Connector:Conn_01x06_Male
- added J_LAN1: RJ45_Amphenol_LMJ1998824110DL1T39J, Greels footprint library:RJ45_Amphenol_LMJ1998824110DL1T39J, symbol Greels symbol library:RJ45_Amphenol_LMJ1998824110DL1T39J
- added L11: 2.2 uH, Greels footprint library:DJNR4018, symbol Device:L
- added Q2, Q3: BC817, Package_TO_SOT_SMD:SOT-23, symbol Transistor_BJT:BC817
- added R29, R35: 220 R, Resistor_SMD:R_0603_1608Metric, symbol Device:R
- added R30: 0 R, Resistor_SMD:R_0603_1608Metric, symbol Device:R
- added R31, R32, R33, R34: 49.9 R, Resistor_SMD:R_0603_1608Metric, symbol Device:R
- added R36: 12.1 k, Resistor_SMD:R_0603_1608Metric, symbol Device:R
- added R37, R38, R39, R40, R42, R43, R44, R45: 2.2 k, Resistor_SMD:R_0603_1608Metric, symbol Device:R
- added R41: 4.7 k, Resistor_SMD:R_0603_1608Metric, symbol Device:R
- added R46: 1k nebo 4k7, Resistor_SMD:R_0603_1608Metric, symbol Device:R
- added R47: NA / 4k7, Resistor_SMD:R_0603_1608Metric, symbol Device:R
- added R48, R49: 4k7, Resistor_SMD:R_0603_1608Metric, symbol Device:R
- added R50, R51: 1k, Resistor_SMD:R_0603_1608Metric, symbol Device:R
- added SW_reset1: SW_Push, Button_Switch_SMD:SW_Push_1P1T_NO_6x6mm_H9.5mm, symbol Switch:SW_Push
- added U7: LAN8710A, Package_DFN_QFN:QFN-32-1EP_5x5mm_P0.5mm_EP3.3x3.3mm_ThermalVias, symbol Interface_Ethernet:LAN8710A
- added U8: ESP32-WROOM-32, RF_Module:ESP32-WROOM-32, symbol Greels_controller_library:ESP32-WROOM-32
Connections:
- new net: R35.1, U7.2 (LED2/~{INTSEL})
- new net: J_LAN1.L3 (LEDG_K), R35.2
- new net: C93.1, R41.2, U7.19 (~{RST})
- new net: Q3.1 (B), R51.2
- new net: C86.1, J_LAN1.R2 (TCT), J_LAN1.R5 (RCT), R30.2
- new net: Q2.1 (B), R50.2
- new net: R37.1, U7.9 (RXD2/~{RMIISEL})
- new net: R40.1, U7.13 (RXER/RXD4/~{PHYAD0})
- new net: C90.1, C91.1, U7.6 (VDDCR)
- new net: R29.2, U7.3 (LED1/~{REGOFF})
- new net: R36.1, U7.32 (RBIAS)
- new net: R39.1, U7.7 (RXCLK/~{PHYAD1})
- new net: R38.1, U7.8 (RXD3/~{PHYAD2})
- new net: J_LAN1.L1 (LEDY_A), R29.1
- new net +3V3: C85.1, C92.2, C95.2, L11.2, R37.2, R41.1, R42.2, R43.2, R44.1, R45.1, R46.1, R47.2, R48.1, R49.1, U7.12 (VDDIO), U8.2 (VDD)
- new net +3V3LAN_ISO: C87.1, C88.1, C89.1, J_LAN1.L4 (LEDG_A), L11.1, R30.1, R31.1, R32.1, R33.1, R34.1, U7.1 (VDD2A), U7.27 (VDD1A)
- new net 5V_ESP: J6.1 (Pin_1)
- new net DTR: J6.5 (Pin_5), Q3.2 (E), R50.1
- new net ESP_EN: C94.1, Q2.3 (C), R46.2, SW_reset1.2, U8.3 (EN)
- new net GND: C85.2, C86.2, C87.2, C88.2, C89.2, C90.2, C91.2, C92.1, C93.2, C94.2, C95.1, J6.6 (Pin_6), J_LAN1.L2 (LEDY_K), J_LAN1.R8 (GND), R36.2, R38.2, R39.2, R40.2, SW_reset1.1, U7.24 (TXD2), U7.25 (TXD3), U7.33 (VSS), U8.1 (GND), U8.15 (GND), U8.38 (GND), U8.39 (GND)
- new net GPI34: U8.6 (IO34)
- new net GPI35: U8.7 (IO35)
- new net GPI36: U8.4 (IO36)
- new net GPI39: U8.5 (IO39)
- new net GPIO0: Q3.3 (C), R47.1, U8.25 (IO0)
- new net GPIO12\PHY_PWR: U8.14 (IO12)
- new net GPIO13: U8.16 (IO13)
- new net GPIO14: U8.13 (IO14)
- new net GPIO15: U8.23 (IO15)
- new net GPIO16: U8.27 (IO16)
- new net GPIO17\EMAC_CLK: U7.5 (XTAL1/CLKIN), U8.28 (IO17)
- new net GPIO18\MDIO(RMII): R43.1, U7.16 (MDIO), U8.30 (IO18)
- new net GPIO19\EMAC_TXD0(RMII): U7.22 (TXD0), U8.31 (IO19)
- new net GPIO1\U0TXD: D4.1 (K), U8.35 (TXD0/IO1)
- new net GPIO21\EMAC_TX_EN(RMII): U7.21 (TXEN), U8.33 (IO21)
- new net GPIO22\EMAC_TXD1(RMII): U7.23 (TXD1), U8.36 (IO22)
- new net GPIO23\MDC(RMII): U7.17 (MDC), U8.37 (IO23)
- new net GPIO25\EMAC_RXD0(RMII): R45.2, U7.11 (RXD0/~{MODE0}), U8.10 (IO25)
- new net GPIO26\EMAC_RXD1(RMII): R44.2, U7.10 (RXD1/~{MODE1}), U8.11 (IO26)
- new net GPIO27\EMAC_RX_CRS_DV: R42.1, U7.15 (COL/CRS_DV/~{MODE2}), U8.12 (IO27)
- new net GPIO2\ONEWIRE: U8.24 (IO2)
- new net GPIO3\U0RXD: D3.2 (A), U8.34 (RXD0/IO3)
- new net GPIO4\RGB_LED: U8.26 (IO4)
- new net GPIO5\SPI_CS: U8.29 (IO5)
- new net I2C_SCL: R48.2, U8.8 (IO32)
- new net I2C_SDA: R49.2, U8.9 (IO33)
- new net RD+: J_LAN1.R4 (RD+), R32.2, U7.31 (RXP)
- new net RD-: J_LAN1.R6 (RD-), R31.2, U7.30 (RXN)
- new net RTS: J6.4 (Pin_4), Q2.2 (E), R51.1
- new net RX: D3.1 (K), J6.2 (Pin_2)
- new net TD+: J_LAN1.R1 (TD+), R34.2, U7.29 (TXP)
- new net TD-: J_LAN1.R3 (TD-), R33.2, U7.28 (TXN)
- new net TX: D4.2 (A), J6.3 (Pin_3)
- no-connect marks 0 -> 12
Other:
- note added: "ESP WROOM MODULE"
- note added: "Programming interface"
