File: ManiAmpPCB/power.kicad_sch (KiCad schematic)
At the start: 0 parts

Commit message: Schematics WiP
Parts:
- added C48 (x4), C50: 100 n, symbol Device:C
- added C49 (x3), C51: 10 u, symbol Device:C
- added C49: 1 u, symbol Device:C
- added C70, C71: 10 uF 50V, Capacitor_SMD:C_1206_3216Metric, symbol Device:C
- added C72: 10 nF, Capacitor_SMD:C_0603_1608Metric, symbol Device:C
- added C73, C76, C79, C82: 100 nF, Capacitor_SMD:C_0603_1608Metric, symbol Device:C
- added C74: 2.7 nF, Capacitor_SMD:C_0603_1608Metric, symbol Device:C
- added C75: open, Capacitor_SMD:C_0603_1608Metric, symbol Device:C
- added C77, C78, C80, C83, C84: 22 uF, Capacitor_SMD:C_0805_2012Metric, symbol Device:C
- added C81: 22 pF, Capacitor_SMD:C_0603_1608Metric, symbol Device:C
- added CP1: 100 uF, Capacitor_SMD:CP_Elec_8x10, symbol Device:C_Polarized
- added D2: SS24, Greels footprint library:DO-214AA, symbol Device:D_Schottky
- added F1: Polyfuse, Fuse:Fuse_2920_7451Metric, symbol Device:Polyfuse
- added J5: Conn_01x02_Socket, symbol Connector:Conn_01x02_Socket
- added L10: 2.2 uH, Greels footprint library:DJNR4018, symbol Device:L
- added L9: 3.6 uH, Inductor_SMD:L_Changjiang_FNR6045S, symbol Device:L
- added R22, R26: 10 k, Resistor_SMD:R_0603_1608Metric, symbol Device:R
- added R23: 15 k, Resistor_SMD:R_0603_1608Metric, symbol Device:R
- added R24: 124k 1%, Resistor_SMD:R_0603_1608Metric, symbol Device:R
- added R240: 240 r, symbol Device:R
- added R25, R28: 22.1 k 1%, Resistor_SMD:R_0603_1608Metric, symbol Device:R
- added R27: 100 k 1%, Resistor_SMD:R_0603_1608Metric, symbol Device:R
- added R52: 1.5 k, symbol Device:R
- added R53, R54: 4.7 k, symbol Device:R
- added R_shunt1: 0.05 R, symbol Device:R
- added U10: LM317_SOT-223, Package_TO_SOT_SMD:SOT-223-3_TabPin2, symbol Regulator_Linear:LM317_SOT-223
- added U11: INA219AxD, Package_SO:SOIC-8_3.9x4.9mm_P1.27mm, symbol Sensor_Energy:INA219AxD
- added U4: AP1117-33, Package_TO_SOT_SMD:SOT-223-3_TabPin2, symbol Regulator_Linear:AP1117-33
- added U5: AP64501SP-13, Greels footprint library:SOIC127P600X170-9N, symbol Greels symbol library:AP64501SP-13
- added U6: AP3429, Package_TO_SOT_SMD:TSOT-23-5, symbol Greels symbol library:AP3429
Connections:
- new net: C81.2, R27.2, R28.1, U6.5 (FB)
- new net: F1.1, J5.2 (Pin_2)
- new net: F1.2, R53.1, R_shunt1.1
- new net: C73.1, U5.1 (BST)
- new net: C73.2, L9.1, U5.8 (SW)
- new net: C72.1, U5.4 (SS)
- new net: C75.1, C76.1, C77.1, C78.1, D2.2 (A), L9.2, R24.1
- new net: R240.2, R52.1, U10.1 (ADJ)
- new net: R26.2, U6.1 (EN)
- new net: L10.1, U6.3 (LX)
- new net: C74.1, R23.2
- new net: C49.1, R54.2, U11.7 (IN-)
- new net: C49.2, R53.2, U11.8 (IN+)
- new net: R22.2, U5.3 (EN)
- new net: C75.2, R24.2, R25.1, U5.5 (FB)
- new net: R23.1, U5.6 (COMP)
- new net +3.3VA: C48.1, C49.2, U4.2 (VO)
- new net +3V3: C48.1, C81.1, C82.1, C83.1, C84.1, L10.2, R27.1, U11.5 (VS)
- new net +5V: C50.1, C51.2, C79.1, C80.1, D2.1 (K), R26.1, U4.3 (VI), U6.4 (VIN)
- new net +9V: C48.1, C49.2, R240.1, U10.2 (VO)
- new net +vin: C48.1, C49.2, C70.1, C71.1, CP1.1, R22.1, R54.1, R_shunt1.2, U10.3 (VI), U5.2 (VIN)
- new net GND: C48.2, C48.2, C48.2, C48.2, C49.1, C49.1, C49.1, C50.2, C51.1, C70.2, C71.2, C72.2, C74.2, C76.2, C77.2, C78.2, C79.2, C80.2, C82.2, C83.2, C84.2, CP1.2, J5.1 (Pin_1), R25.2, R28.2, R52.2, U11.1 (A1), U11.2 (A0), U11.6 (GND), U4.1 (GND), U5.7 (GND), U5.9 (EP), U6.2 (GND)
- new net I2C_SCL: U11.4 (SCL)
- new net I2C_SDA: U11.3 (SDA)
